File: bat_board.sch (KiCad schematic (older format))
At the start: 11 parts

Commit message: Work on the schematic
Parts:
- added C? (x3): C_Small, symbol C_Small
- added D? (x2): Led_Small, symbol Led_Small
- added R? (x2): R_Small, symbol R_Small
- added Y?: Crystal_Small, symbol Crystal_Small
Connections:
- net labels added: D, E, F, G, H, I
- wire segments 28 -> 56
- no-connect marks 0 -> 8
Other:
- moved on the sheet: U?
